Commit message: Added gazebo CAM plugin and object model (box)

File: src/custom_codes/urdf/plugin.gazebo.xacro (robot description, xacro)
@@ -1,9 +1,124 @@
 <?xml version="1.0"?>
 <robot xmlns:xacro="http://wiki.ros.org/xacro">
-<gazebo>
-  <plugin name="gazebo_ros_control" filename="libhwi_switch_gazebo_ros_control.so">
-    <robotNamespace></robotNamespace>
-    <robotSimType>cob_gazebo_ros_control/HWISwitchRobotHWSim</robotSimType>
-  </plugin>
-</gazebo>
+  <gazebo>
+    <plugin name="gazebo_ros_control" filename="libhwi_switch_gazebo_ros_control.so">
+      <robotNamespace></robotNamespace>
+      <robotSimType>cob_gazebo_ros_control/HWISwitchRobotHWSim</robotSimType>
+    </plugin>
+  </gazebo>
+  <!-- <gazebo reference="robotiq_85_left_inner_knuckle_link">
+    <material>Gazebo/Black</material>
+    <turnGravityOff>true</turnGravityOff>
+    <implicitSpringDamper>1</implicitSpringDamper>
+    <kp>100000.0</kp>
+    <kd>1.0</kd>
+    <mu1>10.0</mu1>
+    <mu2>0.1</mu2>
+    <fdir1>0 0 1</fdir1>
+    <minDepth>0.01</minDepth>
+  </gazebo>
+  <gazebo reference="robotiq_85_left_finger_tip_link">
+    <material>Gazebo/Black</material>
+    <turnGravityOff>true</turnGravityOff>
+    <implicitSpringDamper>1</implicitSpringDamper>
+    <kp>100000.0</kp>
+    <kd>1.0</kd>
+    <mu1>10.0</mu1>
+    <mu2>0.1</mu2>
+    <fdir1>0 0 1</fdir1>
+    <minDepth>0.01</minDepth>
+  </gazebo>
+  <gazebo reference="robotiq_85_left_knuckle_link">
+    <material>Gazebo/Black</material>
+    <turnGravityOff>true</turnGravityOff>
+    <implicitSpringDamper>1</implicitSpringDamper>
+    <kp>100000.0</kp>
+    <kd>1.0</kd>
+    <mu1>10.0</mu1>
+    <mu2>0.1</mu2>
+    <fdir1>0 0 1</fdir1>
+    <minDepth>0.01</minDepth>
+  </gazebo>
+  <gazebo reference="robotiq_85_right_inner_knuckle_link">
+    <material>Gazebo/Black</material>
+    <turnGravityOff>true</turnGravityOff>
+    <implicitSpringDamper>1</implicitSpringDamper>
+    <kp>100000.0</kp>
+    <kd>1.0</kd>
+    <mu1>10.0</mu1>
+    <mu2>0.1</mu2>
+    <fdir1>0 0 1</fdir1>
+    <minDepth>0.01</minDepth>
+  </gazebo>
+  <gazebo reference="robotiq_85_right_finger_tip_link">
+    <material>Gazebo/Black</material>
+    <turnGravityOff>true</turnGravityOff>
+    <implicitSpringDamper>1</implicitSpringDamper>
+    <kp>100000.0</kp>
+    <kd>1.0</kd>
+    <mu1>10.0</mu1>
+    <mu2>0.1</mu2>
+    <fdir1>0 0 1</fdir1>
+    <minDepth>0.01</minDepth>
+  </gazebo>
+  <gazebo reference="robotiq_85_right_knuckle_link">
+    <material>Gazebo/Black</material>
+    <turnGravityOff>true</turnGravityOff>
+    <implicitSpringDamper>1</implicitSpringDamper>
+    <kp>100000.0</kp>
+    <kd>1.0</kd>
+    <mu1>10.0</mu1>
+    <mu2>0.1</mu2>
+    <fdir1>0 0 1</fdir1>
+    <minDepth>0.01</minDepth>
+  </gazebo> -->
+  <gazebo reference="box_link">
+    <implicitSpringDamper>1</implicitSpringDamper>
+    <kp>100000.0</kp>
+    <kd>1.0</kd>
+    <mu1>10.0</mu1>
+    <mu2>0.1</mu2>
+    <fdir1>1 0 0</fdir1>
+    <minDepth>0.01</minDepth>
+  </gazebo>
+  <!-- camera -->
+  <gazebo reference="CAM_support_link">
+    <sensor type="camera" name="camera1">
+      <update_rate>30.0</update_rate>
+      <camera name="head">
+        <horizontal_fov>1.3962634</horizontal_fov>
+        <image>
+          <width>800</width>
+          <height>800</height>
+          <format>R8G8B8</format>
+        </image>
+        <clip>
+          <near>0.02</near>
+          <far>300</far>
+        </clip>
+        <noise>
+          <type>gaussian</type>
+          <!-- Noise is sampled independently per pixel on each frame.
+               That pixel's noise value is added to each of its color
+               channels, which at that point lie in the range [0,1]. -->
+          <mean>0.0</mean>
+          <stddev>0.007</stddev>
+        </noise>
+      </camera>
+      <plugin name="camera_controller" filename="libgazebo_ros_camera.so">
+        <alwaysOn>true</alwaysOn>
+        <updateRate>0.0</updateRate>
+        <cameraName>ur5/camera1</cameraName>
+        <imageTopicName>image_raw</imageTopicName>
+        <cameraInfoTopicName>camera_info</cameraInfoTopicName>
+        <frameName>camera_link</frameName>
+        <hackBaseline>0.07</hackBaseline>
+        <distortionK1>0.0</distortionK1>
+        <distortionK2>0.0</distortionK2>
+        <distortionK3>0.0</distortionK3>
+        <distortionT1>0.0</distortionT1>
+        <distortionT2>0.0</distortionT2>
+      </plugin>
+    </sensor>
+  </gazebo>
 </robot>

File: src/custom_codes/urdf/ur5_with_cam.urdf.xacro (robot description, xacro)
@@ -30,7 +30,10 @@
   <!-- CAM SUPPORT CODE -->
   <!-- o wrist 2 fica 0.09465 m abaixo de wrist 3 (-0.0445+0.09465)-->
+  <!-- Its position is relative to its own (Caution: treat as inverse direction)-->
+  <!-- Its orientation is relative to the previous frame -->
   <link name="CAM_support_link">
     <visual>
-      <origin rpy="1.57 3.14 0" xyz="0.002 -0.023 0.13915"/>
+      <!-- The cam is rotated 14 degrees (0.24rad) through the yaw axis -->
+      <origin rpy="${1.57 - 0.244} ${3.14} -1.57" xyz="${0.002 - 0.03} ${-0.023 + 0.03 - 0.01} ${0.13915-0.205}"/>
       <geometry>
         <mesh filename="package://custom_codes/models/cam_support/CAM_support.STL" scale="0.001 0.001 0.001"/>
@@ -42,5 +45,10 @@
   </link>
   <joint name="CAM_support_joint" type="fixed">
-    <origin rpy="0 0 0" xyz="0.0 0.0 0.0"/>
+    <!-- Its position is relative to the previous link -->
+    <!-- Its orientation is relative to its own -->
+    <!-- When you decrease the x component - the cam support move to the left -->
+    <!-- When you decrease the y component - the cam support move backwards -->
+    <!-- z - 30 -->
+    <origin rpy="0 ${0.244} 1.57" xyz="${-0.021 + 0.03 - 0.01} ${-0.027 + 0.03 + 0.015} ${0.205 - 0.0086}"/>
     <parent link="wrist_2_link"/>
     <child link="CAM_support_link"/>
@@ -70,5 +78,5 @@
       </inertial>
     </link>
-    <joint name="lar_table_great_joint" type="fixed">
+  <joint name="lar_table_great_joint" type="fixed">
       <origin rpy="0 0 0" xyz="0 0 0.0"/>
       <parent link="world"/>
