Commit message: Velocity control configuration in gazebo and LAR model

File: src/custom_codes/urdf/ur5_with_cam.urdf.xacro (robot description, xacro)
@@ -1,49 +1,25 @@
 <?xml version="1.0"?>
-<robot xmlns:xacro="http://wiki.ros.org/xacro"
-       name="ur5" >
+<robot xmlns:xacro="http://wiki.ros.org/xacro" name="ur5">
   <xacro:arg name="transmission_hw_interface" default="hardware_interface/PositionJointInterface"/>
+  <xacro:arg name="robot_pose" default="0.0"/>
+  <xacro:arg name="load_table" default="false"/>
   <!-- Gazebo plugin -->
-  <xacro:include filename="$(find custom_codes)/urdf/plugin.gazebo.xacro" />
+  <xacro:include filename="$(find custom_codes)/urdf/plugin.gazebo.xacro"/>
   <!-- Robotiq gripper -->
-  <xacro:include filename="$(find robotiq_description)/urdf/robotiq_85_gripper.urdf.xacro" />
+  <xacro:include filename="$(find robotiq_description)/urdf/robotiq_85_gripper.urdf.xacro"/>
   <!-- ur5 -->
-  <xacro:include filename="$(find ur_description)/urdf/ur5.urdf.xacro" />
+  <xacro:include filename="$(find custom_codes)/urdf/ur5.urdf.xacro"/>
   <!-- It is necessary to change the hardware interface on the fly -->
-  <xacro:include filename="$(find custom_codes)/urdf/ur5.transmission.xacro" />
+  <xacro:include filename="$(find custom_codes)/urdf/ur5.transmission.xacro"/>
   <!-- arm -->
-  <xacro:ur5_robot prefix="" joint_limited="false"
-    transmission_hw_interface="$(arg transmission_hw_interface)"
-  />
-  <link name="world" />
+  <xacro:ur5_robot prefix="" joint_limited="false" transmission_hw_interface="$(arg transmission_hw_interface)"/>
+  <link name="world"/>
   <joint name="world_joint" type="fixed">
-    <parent link="world" />
-    <child link = "base_link" />
-    <origin xyz="0.0 0.0 0.0" rpy="0.0 0.0 0.0" />
-  </joint>
-  <link name="CAM_support">
-    <visual>
-      <!-- o wrist 2 fica 0.09465 m abaixo de wrist 3 (-0.0445+0.09465)-->
-      <origin rpy="1.57 3.14 0" xyz="0.002 -0.023 0.13915"/>
-      <geometry>
-        <mesh filename="package://custom_codes/STL_Files/CAM_support.STL" scale="0.001 0.001 0.001"/>
-      </geometry>
-      <material name="LightGrey">
-        <color rgba="0.91 0.91 0.88 1.0"/>
-      </material>
-    </visual>
-  </link>
-  <joint name="CAM_support_joint" type="fixed">
-   <origin rpy="0 0 0" xyz="0.0 0.0 0.0"/>
-   <parent link="wrist_2_link"/>
-   <child link="CAM_support"/>
-  </joint>
-  <link name="d435_realsense" />
-  <joint name="wrist3_camera" type="fixed">
-    <parent link="wrist_3_link" />
-    <child link = "d435_realsense" />
-    <origin xyz="0.0 0.0 0.0" rpy="0.0 0.0 0.0" />
+    <parent link="world"/>
+    <child link="base_link"/>
+    <origin xyz="0.0 0.0 $(arg robot_pose)" rpy="0.0 0.0 0.0"/>
   </joint>
   <!-- Frame coincident with all-zeros TCP on UR controller -->
-  <xacro:property name="tool0_offset" value="0.15" />
+  <xacro:property name="tool0_offset" value="0.15"/>
   <link name="grasping_link"/>
   <joint name="ur5_joint_grasping_frame" type="fixed">
@@ -52,9 +28,64 @@
     <child link="grasping_link"/>
   </joint>
-  <!-- GRIPPER CODE -->
+  <!-- CAM SUPPORT CODE -->
+  <!-- o wrist 2 fica 0.09465 m abaixo de wrist 3 (-0.0445+0.09465)-->
+  <link name="CAM_support_link">
+    <visual>
+      <origin rpy="1.57 3.14 0" xyz="0.002 -0.023 0.13915"/>
+      <geometry>
+        <mesh filename="package://custom_codes/models/cam_support/CAM_support.STL" scale="0.001 0.001 0.001"/>
+      </geometry>
+      <material name="Cyan">
+        <color rgba="0.91 0.91 0.88 1.0"/>
+      </material>
+    </visual>
+  </link>
+  <joint name="CAM_support_joint" type="fixed">
+    <origin rpy="0 0 0" xyz="0.0 0.0 0.0"/>
+    <parent link="wrist_2_link"/>
+    <child link="CAM_support_link"/>
+  </joint>
+  <!-- TABLE -->
+  <xacro:if value="$(arg load_table)">
+    <link name="lar_table_great_link">
+      <visual>
+        <origin rpy="0 0 1.57" xyz="-0.6 0 0.420"/>
+        <geometry>
+          <mesh filename="package://custom_codes/models/lar_table_great/lar_table_great.stl" scale="0.025 0.025 0.025"/>
+        </geometry>
+        <material name="LightGrey">
+          <color rgba="0.65 0.47 0.19 1.0"/>
+        </material>
+      </visual>
+      <collision name="lar_table_great__collisions">
+        <origin rpy="0 0 0" xyz="0 0 0.445"/>
+        <geometry>
+          <mesh filename="package://custom_codes/models/lar_table_great/lar_table_great.stl" scale="0.025 0.025 0.025"/>
+        </geometry>
+      </collision>
+      <inertial>
+        <mass value="25"/>
+        <origin rpy="0 0 0" xyz="0 0 0"/>
+        <inertia ixx="1" ixy="0" ixz="0" iyy="1" iyz="0" izz="1"/>
+      </inertial>
+    </link>
+    <joint name="lar_table_great_joint" type="fixed">
+      <origin rpy="0 0 0" xyz="0 0 0.0"/>
+      <parent link="world"/>
+      <child link="lar_table_great_link"/>
+    </joint>
+  </xacro:if>
+  <!-- REALSENSE CODE -->
+  <link name="d435_realsense"/>
+  <joint name="wrist3_camera" type="fixed">
+    <parent link="wrist_3_link"/>
+    <child link="d435_realsense"/>
+    <origin xyz="0.0 0.0 0.0" rpy="0.0 0.0 0.0"/>
+  </joint>
+  <!-- GAZEBO ROBOTIQ CODE -->
   <link name="robotiq_coupler">
     <visual>
       <geometry>
-        <mesh filename="package://robotiq_description/meshes/robotiq_85_coupler.stl" />
+        <mesh filename="package://robotiq_description/meshes/robotiq_85_coupler.stl"/>
       </geometry>
       <material name="flat_black"/>
@@ -62,16 +93,15 @@
     <collision>
       <geometry>
-        <mesh filename="package://robotiq_description/meshes/robotiq_85_coupler.stl" />
+        <mesh filename="package://robotiq_description/meshes/robotiq_85_coupler.stl"/>
       </geometry>
     </collision>
     <inertial>
-      <origin xyz="2.073e-05   1.45286e-03  -1.1049e-03" rpy="0 0 0" />
-      <mass value="0.168" />
-      <inertia ixx="6.69695624e-05" ixy="5.21511788e-09" ixz="-2.74383009e-08"
-               iyy="7.85088161e-05" iyz="5.41105193e-07" izz="1.41819717e-04"/>
+      <origin xyz="2.073e-05   1.45286e-03  -1.1049e-03" rpy="0 0 0"/>
+      <mass value="0.168"/>
+      <inertia ixx="6.69695624e-05" ixy="5.21511788e-09" ixz="-2.74383009e-08" iyy="7.85088161e-05" iyz="5.41105193e-07" izz="1.41819717e-04"/>
     </inertial>
-</link>
-    <joint name="robotiq_coupler_joint" type="fixed">
-    <origin xyz="0 0 0.004" rpy="0 0 ${-pi/2.0}" />
+  </link>
+  <joint name="robotiq_coupler_joint" type="fixed">
+    <origin xyz="0 0 0.004" rpy="0 0 ${-pi/2.0}"/>
     <parent link="tool0"/>
     <child link="robotiq_coupler"/>
@@ -81,10 +111,8 @@
     <mu2>0.9</mu2>
     <material>Gazebo/FlatBlack</material>
-</gazebo>
- <!-- Attach the robotiq 85 gripper -->
-  <xacro:robotiq_85_gripper prefix="" parent="robotiq_coupler" >
+  </gazebo>
+  <xacro:robotiq_85_gripper prefix="" parent="robotiq_coupler">
     <origin xyz="0 0 0.004" rpy="0 ${-pi/2} ${pi}"/>
   </xacro:robotiq_85_gripper>
-  <!-- Gazebo FT sensor plugin -->
   <gazebo reference="wrist_3_joint">
     <provideFeedback>true</provideFeedback>
@@ -98,5 +126,4 @@
     </plugin>
   </gazebo>
-  <!-- Gazebo grasping plugin -->
   <gazebo>
     <gripper name="gazebo_gripper">
@@ -110,4 +137,4 @@
       <palm_link>robotiq_85_base_link</palm_link>
     </gripper>
-</gazebo>
+  </gazebo>
 </robot>

Commit message: ar_track_alvar can now be detected by the gazebo cam plugin

File: src/custom_codes/urdf/ur5_with_cam.urdf.xacro (robot description, xacro)
@@ -27,4 +27,11 @@
     <parent link="tool0"/>
     <child link="grasping_link"/>
+  </joint>
+  <!-- This frame is placed in the same position as the box inserted in Gazebo in order to be visualized in RVIZ (just for comparison) -->
+  <link name="reference_link"/>
+  <joint name="reference_frame" type="fixed">
+    <origin xyz="-0.5 0.1 0.05" rpy="0 0 -0.6"/>
+    <parent link="base_link"/>
+    <child link="reference_link"/>
   </joint>
   <!-- CAM SUPPORT CODE -->
